File: HW_roggeluc_linortho/HW_roggeluc_linortho.kicad_pcb (KiCad board)
At the start: 2 copper layers, 63.5 x 118.1 mm, 59 parts, among them J1 USB_B_Mini, P1 type="R" model="Conn_01x32_Fe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, P2 type="R" model="Conn_01x32_Fe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, Q1 BSS316N, SW1 type="R" model="SW_Push" lib=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, U1 MCP6002-xSN, U2 MCP6002-xSN, U3 SiP32508, U4 LD1117S33TR_SOT223, U5 type="R" model="DRV5053_SMD" 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, U6 type="R" model="DRV5053_THT" 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, U7 MCP6002-xSN, Y1 OpenLog, Y2 Radar K-LC5-RFB-00C

Commit message: lol
Parts:
- removed C2, C3: 100n, Capacitor_SMD:C_0805_2012Metric_Pad1.18x1.45mm_HandSolder
- removed C4: 100uF, Capacitor_SMD:C_1206_3216Metric_Pad1.33x1.80mm_HandSolder
- removed C6: 10uF, Capacitor_SMD:C_0805_2012Metric_Pad1.18x1.45mm_HandSolder
- removed C8, C9: 100nF, Capacitor_SMD:C_0805_2012Metric_Pad1.18x1.45mm_HandSolder
- removed LED1: LEDblue, LED_SMD:LED_1206_3216Metric_Pad1.42x1.75mm_HandSolder
- removed LED2: LEDgreen, LED_SMD:LED_1206_3216Metric_Pad1.42x1.75mm_HandSolder
- removed Lconn1, Lconn2: Conn_01x02_Male, Connector_PinHeader_2.54mm:PinHeader_1x02_P2.54mm_Vertical
- removed P1, P2: type="R" model="Conn_01x32_Female" lib="", Connector_PinSocket_2.54mm:PinSocket_1x32_P2.54mm_Vertical
- removed R1: 10k, Resistor_SMD:R_0805_2012Metric_Pad1.20x1.40mm_HandSolder
- removed R10: 47, Resistor_SMD:R_0805_2012Metric_Pad1.20x1.40mm_HandSolder
- removed R12, R14: 100, Resistor_SMD:R_0805_2012Metric_Pad1.20x1.40mm_HandSolder
- removed R13, R2, R4, R6, R8: 1k, Resistor_SMD:R_0805_2012Metric_Pad1.20x1.40mm_HandSolder
- removed R3: 12k, Resistor_SMD:R_0805_2012Metric_Pad1.20x1.40mm_HandSolder
- removed R5: 220k, Resistor_SMD:R_0805_2012Metric_Pad1.20x1.40mm_HandSolder
- removed R7: 100k, Resistor_SMD:R_0805_2012Metric_Pad1.20x1.40mm_HandSolder
- removed R9: 22, Resistor_SMD:R_0805_2012Metric_Pad1.20x1.40mm_HandSolder
- removed SD1: SD103AWS, Diode_SMD:D_SOD-323_HandSoldering
- removed TP3: pad_left, TestPoint:TestPoint_Loop_D2.60mm_Drill1.6mm_Beaded
- removed TP5: coil_left, TestPoint:TestPoint_Loop_D2.60mm_Drill1.6mm_Beaded
- removed the U3 at (115.1, 67.6)
- removed U5: type="R" model="DRV5053_SMD" lib="", Package_TO_SOT_SMD:SOT-23
- removed U6: type="R" model="DRV5053_THT" lib="", HW_template:TO-92Flat_wide
- removed Y1: OpenLog, Connector_PinHeader_2.54mm:PinHeader_1x06_P2.54mm_Vertical
- removed Y2: Radar K-LC5-RFB-00C, HW_template:Radar_K-LC5
- added BT1: BH-18650-PC, BH-18650-PC:BAT_BH-18650-PC, B.Cu at (74.5, 79.5)
- added C11: 100n, Capacitor_SMD:C_0805_2012Metric_Pad1.18x1.45mm_HandSolder, F.Cu at (87.2, 106.9)
- added C12: 100n, Capacitor_SMD:C_0805_2012Metric_Pad1.18x1.45mm_HandSolder, F.Cu at (92.7, 75.4)
- added C13: 100n, Capacitor_SMD:C_0805_2012Metric_Pad1.18x1.45mm_HandSolder, F.Cu at (55.5, 95.0)
- added C14: 100n, Capacitor_SMD:C_0805_2012Metric_Pad1.18x1.45mm_HandSolder, F.Cu at (83.7, 106.9)
- added C15: 100n, Capacitor_SMD:C_0805_2012Metric_Pad1.18x1.45mm_HandSolder, F.Cu at (84.2, 84.9)
- added C16: 100n, Capacitor_SMD:C_0805_2012Metric_Pad1.18x1.45mm_HandSolder, F.Cu at (62.0, 107.0)
- added C17: 100n, Capacitor_SMD:C_0805_2012Metric_Pad1.18x1.45mm_HandSolder, F.Cu at (65.5, 107.0)
- added C18: 100n, Capacitor_SMD:C_0805_2012Metric_Pad1.18x1.45mm_HandSolder, F.Cu at (62.5, 85.0)
- added C19: 100n, Capacitor_SMD:C_0805_2012Metric_Pad1.18x1.45mm_HandSolder, F.Cu at (72.0, 75.5)
- added C20: 100n, Capacitor_SMD:C_0805_2012Metric_Pad1.18x1.45mm_HandSolder, F.Cu at (187.1, 25.0)
- added C21: 100n, Capacitor_SMD:C_0805_2012Metric_Pad1.18x1.45mm_HandSolder, F.Cu at (89.2, 75.4)
- added C22: 100n, Capacitor_SMD:C_0805_2012Metric_Pad1.18x1.45mm_HandSolder, F.Cu at (68.0, 75.5)
- added C23: 10uF, Capacitor_SMD:C_0805_2012Metric_Pad1.18x1.45mm_HandSolder, F.Cu at (57.5, 120.9)
- added C24: 10nF, Capacitor_SMD:C_0805_2012Metric_Pad1.18x1.45mm_HandSolder, F.Cu at (61.0, 121.0)
- added C25: 10uF, Capacitor_SMD:C_0805_2012Metric_Pad1.18x1.45mm_HandSolder, F.Cu at (60.5, 155.5)
- added C26: 10uF, Capacitor_SMD:C_0805_2012Metric_Pad1.18x1.45mm_HandSolder, F.Cu at (186.2, 121.2)
- added C27: 10uF, Capacitor_SMD:C_0805_2012Metric_Pad1.18x1.45mm_HandSolder, F.Cu at (46.5, 126.4)
- added C28: 10uF, Capacitor_SMD:C_0805_2012Metric_Pad1.18x1.45mm_HandSolder, F.Cu at (186.2, 124.3)
- added C29: 10uF, Capacitor_SMD:C_0805_2012Metric_Pad1.18x1.45mm_HandSolder, F.Cu at (186.2, 127.3)
- added C30: 10uF, Capacitor_SMD:C_0805_2012Metric_Pad1.18x1.45mm_HandSolder, F.Cu at (186.2, 130.3)
- added CHARGE1: LEDcharge, LED_SMD:LED_1206_3216Metric_Pad1.42x1.75mm_HandSolder, F.Cu at (85.0, 162.5)
- added COMPLETE1: LEDcompl, LED_SMD:LED_1206_3216Metric_Pad1.42x1.75mm_HandSolder, F.Cu at (81.0, 162.5)
- added J2: USB_B_Mini, Connector_USB:USB_Mini-B_Lumberg_2486_01_Horizontal, F.Cu at (70.0, 158.4)
- added P3: DIN41612_02x32_AB, Connector_PinSocket_2.54mm:PinSocket_2x32_P2.54mm_Vertical, F.Cu at (98.0, 119.9)
- added P4: DIN41612_02x32_AB, Connector_PinSocket_2.54mm:PinSocket_2x32_P2.54mm_Vertical, F.Cu at (46.5, 120.0)
- added POWER1: LEDpower, LED_SMD:LED_1206_3216Metric_Pad1.42x1.75mm_HandSolder, F.Cu at (89.0, 162.5)
- added Q10: Si2319CDS, Package_TO_SOT_SMD:SOT-23, F.Cu at (221.1, 56.5)
- added Q2: BSS316N, Package_TO_SOT_SMD:SOT-23, F.Cu at (84.7, 75.4)
- added Q3: BSS316N, Package_TO_SOT_SMD:SOT-23, F.Cu at (64.0, 75.4)
- added Q4: BSS316N, Package_TO_SOT_SMD:SOT-23, F.Cu at (181.4, 116.1)
- added Q5: BSS316N, Package_TO_SOT_SMD:SOT-23, F.Cu at (181.4, 120.8)
- added Q6: BSS316N, Package_TO_SOT_SMD:SOT-23, F.Cu at (181.4, 125.4)
- added Q9: Si2319CDS, Package_TO_SOT_SMD:SOT-23, F.Cu at (181.4, 130.0)
- added R26: 1k, Resistor_SMD:R_0805_2012Metric_Pad1.20x1.40mm_HandSolder, F.Cu at (90.7, 106.9)
- added R27: 1k, Resistor_SMD:R_0805_2012Metric_Pad1.20x1.40mm_HandSolder, F.Cu at (77.7, 84.9)
- added R28: 1k, Resistor_SMD:R_0805_2012Metric_Pad1.20x1.40mm_HandSolder, F.Cu at (77.2, 101.9)
- added R29: 1k, Resistor_SMD:R_0805_2012Metric_Pad1.20x1.40mm_HandSolder, F.Cu at (80.2, 106.9)
- added R30: 1k, Resistor_SMD:R_0805_2012Metric_Pad1.20x1.40mm_HandSolder, F.Cu at (83.2, 89.6)
- added R31: 1k, Resistor_SMD:R_0805_2012Metric_Pad1.20x1.40mm_HandSolder, F.Cu at (80.7, 84.9)
- added R32: 1k, Resistor_SMD:R_0805_2012Metric_Pad1.20x1.40mm_HandSolder, F.Cu at (56.0, 102.0)
- added R33: 1k, Resistor_SMD:R_0805_2012Metric_Pad1.20x1.40mm_HandSolder, F.Cu at (58.5, 107.0)
- added R34: 1k, Resistor_SMD:R_0805_2012Metric_Pad1.20x1.40mm_HandSolder, F.Cu at (69.0, 107.0)
- added R35: 1k, Resistor_SMD:R_0805_2012Metric_Pad1.20x1.40mm_HandSolder, F.Cu at (61.5, 90.5)
- added R36: 1k, Resistor_SMD:R_0805_2012Metric_Pad1.20x1.40mm_HandSolder, F.Cu at (59.0, 84.9)
- added R37: 1k, Resistor_SMD:R_0805_2012Metric_Pad1.20x1.40mm_HandSolder, F.Cu at (56.0, 85.0)
- added R38: 1k, Resistor_SMD:R_0805_2012Metric_Pad1.20x1.40mm_HandSolder, F.Cu at (172.7, 14.9)
- added R39: 10k, Resistor_SMD:R_0805_2012Metric_Pad1.20x1.40mm_HandSolder, F.Cu at (79.7, 75.4)
- added R40: 10k, Resistor_SMD:R_0805_2012Metric_Pad1.20x1.40mm_HandSolder, F.Cu at (59.0, 75.5)
- added R41: 1k, Resistor_SMD:R_0805_2012Metric_Pad1.20x1.40mm_HandSolder, F.Cu at (85.0, 156.0)
- added R42: 1k, Resistor_SMD:R_0805_2012Metric_Pad1.20x1.40mm_HandSolder, F.Cu at (81.0, 156.0)
- added R43: 30.1k, Resistor_SMD:R_0805_2012Metric_Pad1.20x1.40mm_HandSolder, F.Cu at (195.8, 115.2)
- added R44: 330, Resistor_SMD:R_0805_2012Metric_Pad1.20x1.40mm_HandSolder, F.Cu at (195.8, 118.2)
- added R45: 2.7k, Resistor_SMD:R_0805_2012Metric_Pad1.20x1.40mm_HandSolder, F.Cu at (195.8, 121.1)
- added R46: 10k, Resistor_SMD:R_0805_2012Metric_Pad1.20x1.40mm_HandSolder, F.Cu at (195.8, 124.0)
- added R47: 51k, Resistor_SMD:R_0805_2012Metric_Pad1.20x1.40mm_HandSolder, F.Cu at (195.8, 127.0)
- added R48: 1k, Resistor_SMD:R_0805_2012Metric_Pad1.20x1.40mm_HandSolder, F.Cu at (200.5, 115.2)
- added R49: 10k, Resistor_SMD:R_0805_2012Metric_Pad1.20x1.40mm_HandSolder, F.Cu at (200.5, 118.2)
- added R50: 10k, Resistor_SMD:R_0805_2012Metric_Pad1.20x1.40mm_HandSolder, F.Cu at (200.5, 121.1)
- added R51: 100k, Resistor_SMD:R_0805_2012Metric_Pad1.20x1.40mm_HandSolder, F.Cu at (200.5, 124.0)
- added TP10: ~, TestPoint:TestPoint_Loop_D2.60mm_Drill1.6mm_Beaded, F.Cu at (-91.5, 138.7)
- added TP11: ~, TestPoint:TestPoint_Loop_D2.60mm_Drill1.6mm_Beaded, F.Cu at (-107.5, 220.3)
- added TP12: ~, TestPoint:TestPoint_Loop_D2.60mm_Drill1.6mm_Beaded, F.Cu at (192.7, 16.0)
- added TP13: ~, TestPoint:TestPoint_Loop_D2.60mm_Drill1.6mm_Beaded, F.Cu at (192.7, 21.0)
- added TP7: CH2, TestPoint:TestPoint_Loop_D2.60mm_Drill1.6mm_Beaded, F.Cu at (-117.6, 220.3)
- added TP8: ~, TestPoint:TestPoint_Loop_D2.60mm_Drill1.6mm_Beaded, F.Cu at (-112.6, 215.2)
- added TP9: ~, TestPoint:TestPoint_Loop_D2.60mm_Drill1.6mm_Beaded, F.Cu at (-137.5, 130.5)
- added U3: AP3012, Package_TO_SOT_SMD:SOT-23-5, F.Cu at (173.7, 40.8)
- added U3: AP9101CK, Package_TO_SOT_SMD:SOT-23-5, F.Cu at (211.4, 129.1)
- added U8: MCP6002-xSN, Package_SO:SOIC-8_3.9x4.9mm_P1.27mm, F.Cu at (62.0, 97.5)
- added Y4: Radar K-LC5-RFB-00C, HW_template:Radar_K-LC5, B.Cu at (70.5, 128.4)
- C1: footprint Capacitor_SMD:C_1206_3216Metric_Pad1.33x1.80mm_HandSolder -> Capacitor_SMD:C_0805_2012Metric_Pad1.18x1.45mm_HandSolder
- J1: value USB_B_Mini -> Micro_SD_Card; footprint Connector_USB:USB_Mini-B_Lumberg_2486_01_Horizontal -> Connector_Card:microSD_HC_Wuerth_693072010801
- L1: value 15mH -> 10 uH; footprint Inductor_SMD:L_Bourns_SRN6045TA -> Inductor_SMD:L_0805_2012Metric_Pad1.15x1.40mm_HandSolder
- R18: value 10k -> 10kOhm
- R19: value 1k -> 10kOhm
- R20: value 12k -> 1k
- SW1: value type="R" model="SW_Push" lib="" -> SW_MEC_5G; footprint Button_Switch_SMD:SW_SPST_PTS645 -> Button_Switch_SMD:SW_SPST_EVQQ2
- TP6: value ~ -> CH1
- U1: value MCP6002-xSN -> LM2731XMF; footprint Package_SO:SOIC-8_3.9x4.9mm_P1.27mm -> Package_TO_SOT_SMD:SOT-23-5
- U2: value MCP6002-xSN -> MCP73833-xxx-MF; footprint Package_SO:SOIC-8_3.9x4.9mm_P1.27mm -> Package_DFN_QFN:DFN-10-1EP_3x3mm_P0.5mm_EP1.58x2.35mm
- moved TP6 208.6 mm to (-101.6, 138.7)
- moved TP2 152.7 mm to (155.3, 21.0)
- moved L1 147.0 mm to (191.0, 115.2), turned to 0 degrees
- moved U1 144.2 mm to (211.4, 124.4)
- moved R20 134.5 mm to (191.0, 118.2), turned to 0 degrees
- moved TP1 130.2 mm to (155.3, 16.0)
- moved SD2 117.2 mm to (222.8, 116.0), turned to 0 degrees
- moved U4 106.6 mm to (213.8, 117.9), turned to 0 degrees
- moved R21 101.7 mm to (89.0, 156.0), turned to 90 degrees
- moved U2 83.7 mm to (84.4, 150.1), turned to -90 degrees
- moved R16 82.8 mm to (188.0, 58.1), turned to 0 degrees
- moved TP4 76.5 mm to (51.5, 137.4), turned to 180 degrees
- moved R15 75.1 mm to (188.0, 55.1), turned to 0 degrees
- moved C7 74.8 mm to (186.2, 115.2)
- moved SW1 72.3 mm to (109.1, 28.5)
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Connections:
- C1 pad 1: +3V0 -> +3.3V
- C10 pad 1: +3V0 -> +3.3V
- C7 pad 1: Net-(U4-VO) -> +3.3V
- J1 pad 2: unconnected-(J1-D--Pad2) -> PE4
- J1 pad 3: unconnected-(J1-D+-Pad3) -> PE5
- J1 pad 4: unconnected-(J1-ID-Pad4) -> +3V0
- J1 pad 5: GND -> PE2
- L1 pad 1: coil_left -> Net-(U1-VIN)
- L1 pad 2: GND -> Net-(SD2-A)
- L2 pad 1: coil_right -> unconnected-(L2-Pad1)
- L2 pad 2: GND -> unconnected-(L2-Pad2)
- R17 pad 1: Net-(U4-VO) -> Net-(U2-PROG)
- R18 pad 1: Net-(U7B-+) -> +1V65
- R18 pad 2: Net-(U7A--) -> +3.3V
- R19 pad 1: Net-(U7A--) -> GND
- R19 pad 2: GND -> +1V65
- R20 pad 1: PF8_ -> Net-(U2-THERM)
- R20 pad 2: Net-(U7B--) -> GND
- R21 pad 1: Net-(U7B--) -> Net-(POWER1-K)
- R21 pad 2: GND -> Net-(U2-~{PG})
- SD2 pad 1: GND -> Net-(Q9-S)
- SW1 pad 1: unconnected-(SW1-Pad1) -> Net-(SW1-A-Pad1)
- SW1 pad 2: unconnected-(SW1-Pad2) -> Net-(SW1-A-Pad1)
- TP4 pad 1: PC3 -> +1V65
- TP6 pad 1: PC1_ -> PC4
- U1 pad 1: Net-(U1B-+) -> Net-(SD2-A)
- U1 pad 2: Net-(U1A--) -> GND
- U1 pad 3: coil_right -> Net-(U1-FB)
- U1 pad 4: GND -> Net-(Q6-D)
- U1 pad 5: Net-(U1B-+) -> Net-(U1-VIN)
- U2 pad 1: PF6 -> 5V
- U2 pad 2: Net-(U2A--) -> 5V
- U2 pad 3: pad_left -> Net-(U2-STAT1)
- U2 pad 4: GND -> Net-(U2-STAT2)
- U2 pad 5: pad_right -> GND
- U2 pad 6: Net-(U2B--) -> Net-(U2-PROG)
- U2 pad 7: PC3 -> Net-(U2-~{PG})
- U2 pad 8: +3V0 -> Net-(U2-THERM)
- U4 pad 2: Net-(U4-VO) -> +3.3V
- U4 pad 3: Net-(U4-VI) -> Net-(Q9-S)
- U7 pad 3: coil_left -> Net-(U7A-+)
- U7 pad 7: PF8_ -> Net-(R27-Pad1)
- U7 pad 8: +3V0 -> +3.3V
Routing:
- net +3V0: track 39.4 -> 0.00 mm, vias 6 -> 0
- net pad_right: track 33.2 -> 0.00 mm, vias 2 -> 0
- net +1V65: track 0.00 -> 33.0 mm
- net coil_left: track 32.7 -> 0.00 mm, vias 1 -> 0
- net coil_right: track 31.5 -> 0.00 mm, vias 1 -> 0
- net pad_left: track 31.2 -> 0.00 mm, vias 2 -> 0
- net +3.3V: track 0.00 -> 26.6 mm
- net IF_I: track 0.00 -> 25.3 mm
- net PC5: track 0.00 -> 24.2 mm
- net PF8_: track 24.0 -> 0.00 mm, vias 1 -> 0
- net PC1_: track 24.0 -> 0.00 mm, vias 1 -> 0
- net IF_Q: track 0.00 -> 22.5 mm
- net PC4: track 0.00 -> 21.6 mm
- net PC3: track 20.6 -> 0.00 mm, vias 1 -> 0
- net PF6: track 20.1 -> 0.00 mm, vias 1 -> 0
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- removed copper zone on B.Cu, net GND
- removed copper zone on F.Cu, net GND
- removed copper zone on B.Cu, net pad_left
- removed copper zone on F.Cu, net pad_left
- removed copper zone on B.Cu, net pad_right
- removed copper zone on F.Cu, net pad_right
Other:
- board size 63.5 x 118.1 mm -> 66 x 118 mm
- board text removed: "Sensor-Board: HW template for ET.PM3 = Cable-Monitor and ET.PM4 = Radar-Sensor (c) hhrt@zhaw.ch January 2023"
- board text removed: "The 32 pin connectors are on the bottom side!"
- board text removed: "The GND plates have already been added. Press B to fill, CTRL + B to unfill all plates/zones."

Commit message: PCB ORDERED
Parts:
- removed L2: 15mH, Inductor_SMD:L_Bourns_SRN6045TA
- removed Q9: Si2319CDS, Package_TO_SOT_SMD:SOT-23
- removed R50: 10k, Resistor_SMD:R_0805_2012Metric_Pad1.20x1.40mm_HandSolder
- removed R51: 100k, Resistor_SMD:R_0805_2012Metric_Pad1.20x1.40mm_HandSolder
- removed the U3 at (173.7, 40.8)
- added C31: 1uF, Capacitor_SMD:C_0805_2012Metric_Pad1.18x1.45mm_HandSolder, F.Cu at (103.4, 161.6)
- added CHARGE2: LEDcharge, LED_SMD:LED_1206_3216Metric_Pad1.42x1.75mm_HandSolder, F.Cu at (86.6, 32.3)
- added LS1: SMT-0827-S-HT-R, SMT-0827-S-HT-R:XDCR_SMT-0827-S-HT-R, F.Cu at (46.0, 159.5)
- added Q7: BSS316N, Package_TO_SOT_SMD:SOT-23, F.Cu at (101.7, 149.5)
- added R16: 330, Resistor_SMD:R_0805_2012Metric_Pad1.20x1.40mm_HandSolder, F.Cu at (50.0, 147.0)
- added R52: 100k, Resistor_SMD:R_0805_2012Metric_Pad1.20x1.40mm_HandSolder, F.Cu at (103.0, 165.0)
- added R53: 10k, Resistor_SMD:R_0805_2012Metric_Pad1.20x1.40mm_HandSolder, F.Cu at (101.7, 152.4)
- added R54: 10k, Resistor_SMD:R_0805_2012Metric_Pad1.20x1.40mm_HandSolder, F.Cu at (105.2, 151.9)
- added R55: 1k, Resistor_SMD:R_0805_2012Metric_Pad1.20x1.40mm_HandSolder, F.Cu at (86.5, 37.5)
- added SD3: SS13L, Diode_SMD:D_SMA, F.Cu at (96.7, 156.1)
- added TP14: ~, TestPoint:TestPoint_Loop_D2.60mm_Drill1.6mm_Beaded, F.Cu at (44.5, 144.5)
- added TP16: ~, TestPoint:TestPoint_Loop_D2.60mm_Drill1.6mm_Beaded, F.Cu at (58.5, 129.0)
- added TP17: ~, TestPoint:TestPoint_Loop_D2.60mm_Drill1.6mm_Beaded, F.Cu at (73.0, 154.0)
- added TP18: ~, TestPoint:TestPoint_Loop_D2.60mm_Drill1.6mm_Beaded, F.Cu at (94.5, 126.5)
- added TP19: ~, TestPoint:TestPoint_Loop_D2.60mm_Drill1.6mm_Beaded, F.Cu at (43.0, 138.5)
- added TP20: ~, TestPoint:TestPoint_Loop_D2.60mm_Drill1.6mm_Beaded, F.Cu at (90.0, 132.5)
- J1: moved to B.Cu
- SW1: value SW_MEC_5G -> SW_Push_Dual_x2
- moved TP8 252.9 mm to (93.0, 68.0)
- moved TP11 252.7 mm to (89.5, 62.0)
- moved TP7 244.0 mm to (92.0, 95.5)
- moved TP9 202.5 mm to (59.5, 83.5)
- moved TP2 170.9 mm to (43.9, 150.7)
- moved TP6 165.6 mm to (56.5, 89.5)
- moved R16 165.4 mm to (54.0, 155.0)
- moved R15 163.9 mm to (50.0, 143.5)
- moved Q10 163.4 mm to (97.9, 164.0), turned to 180 degrees
- moved TP10 160.1 mm to (54.0, 72.0)
- moved Q1 156.7 mm to (50.0, 150.6), turned to -90 degrees
- moved U3 153.4 mm to (59.0, 145.9), turned to 90 degrees
- moved SW1 142.6 mm to (57.9, 161.6)
- moved R17 141.8 mm to (73.5, 145.0), turned to 90 degrees
- moved TP13 139.3 mm to (89.5, 114.5)
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- renumbered CHARGE1 to CRG1, COMPLETE1 to FULL1, POWER1 to PWR1
Connections:
- C28 pad 2: Net-(Q9-S) -> Net-(Q10-S)
- C29 pad 2: Net-(Q9-S) -> Net-(Q10-S)
- J1 pad 4: +3V0 -> +3.3V
- P3 pad 1: 5V -> +5V
- P3 pad 2: 5V -> +5V
- P3 pad 27: PB3 -> Enable
- P3 pad 51: PA9 -> LED_ON
- Q1 pad 1: Enable -> Net-(Q1-G)
- Q10 pad 1: unconnected-(Q10-G-Pad1) -> Net-(Q10-G)
- Q10 pad 2: unconnected-(Q10-S-Pad2) -> Net-(Q10-S)
- Q10 pad 3: unconnected-(Q10-D-Pad3) -> +5V
- R15 pad 1: Enable -> PA8
- R43 pad 2: Net-(Q9-S) -> Net-(Q10-S)
- SD2 pad 1: Net-(Q9-S) -> Net-(Q10-S)
- SW1 pad 1: Net-(SW1-A-Pad1) -> Net-(SW1A-C)
- SW1 pad 2: Net-(SW1-A-Pad1) -> PA6
- U4 pad 3: Net-(Q9-S) -> Net-(Q10-S)
- Y4 pad 5: unconnected-(Y4-VCO_in-Pad5) -> fmcw_sig
Routing:
- net +3.3V: track 26.6 -> 227.1 mm, vias 0 -> 13
- net PA6: track 0.00 -> 198.2 mm, vias 0 -> 2
- net PA8: track 0.00 -> 150.5 mm, vias 0 -> 6
- net +5V: track 0.00 -> 147.5 mm, vias 0 -> 6
- net PE4: track 0.00 -> 109.3 mm, vias 0 -> 3
- net +1V65: track 33.0 -> 135.5 mm, vias 0 -> 2
- net PE6: track 0.00 -> 96.8 mm, vias 0 -> 9
- net Net-(U1-VIN): track 0.00 -> 90.8 mm, vias 0 -> 6
- net Net-(Q5-S): track 0.00 -> 88.4 mm, vias 0 -> 4
- net PE2: track 0.00 -> 83.8 mm, vias 0 -> 5
- net PE5: track 0.00 -> 81.9 mm, vias 0 -> 3
- net 5V: track 16.2 -> 97.0 mm, vias 0 -> 6
- net Net-(Q10-S): track 0.00 -> 78.2 mm, vias 0 -> 4
- net fmcw_sig: track 0.00 -> 69.3 mm, vias 0 -> 4
- net Net-(SW1A-C): track 0.00 -> 58.2 mm, vias 0 -> 8
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- added copper zone on B.Cu, net GND
Other:
- board size 66 x 118 mm -> 66 x 138.5 mm
- board text added: "Linortho"
- board text added: "Radar Intrudor detection"
- board text added: "Roggeluc"
- board text added: "ZHAW ET.PM4"
