File: HW_roggeluc_linortho/miscellaneous.kicad_sch (KiCad schematic)
At the start: 28 parts, among them J1 ${SIM.PARAMS}, Q1 BSS316N, SW1 ${SIM.PARAMS}, U3 SiP32508, U4 LD1117S33TR_SOT223, U5 ${SIM.PARAMS}, U6 ${SIM.PARAMS}, Y1 ${SIM.PARAMS}, Y2 ${SIM.PARAMS}

Commit message: OPAMP ANTENNA
Other:
- moved on the sheet: Y2
Changed lines of the file:
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@@
 	(text "The Radar sensor\nwill be used in the\nproject module 4"
 		(exclude_from_sim no)
-		(at 236.22 93.98 0)
+		(at 233.68 99.06 0)
 		(effects
 			(font
@@
 	(wire
 		(pts
-			(xy 237.49 119.38) (xy 238.76 119.38)
+			(xy 234.95 124.46) (xy 236.22 124.46)
 		)
 		(stroke
@@
 	(wire
 		(pts
-			(xy 238.76 115.57) (xy 228.6 115.57)
+			(xy 236.22 120.65) (xy 226.06 120.65)
 		)
 		(stroke
@@
 	(wire
 		(pts
-			(xy 228.6 115.57) (xy 228.6 119.38)
+			(xy 226.06 120.65) (xy 226.06 124.46)
 		)
 		(stroke
@@
 	(wire
 		(pts
-			(xy 228.6 107.95) (xy 238.76 107.95)
+			(xy 226.06 113.03) (xy 236.22 113.03)
 		)
 		(stroke
@@
 	(wire
 		(pts
-			(xy 228.6 104.14) (xy 228.6 107.95)
+			(xy 226.06 109.22) (xy 226.06 113.03)
 		)
 		(stroke
@@
 	(global_label "PA5"
 		(shape input)
-		(at 237.49 119.38 180)
+		(at 234.95 124.46 180)
 		(fields_autoplaced yes)
 		(effects
@@
 		)
 		(property "Intersheetrefs" "${INTERSHEET_REFS}"
-			(at 231.5088 119.3006 0)
+			(at 228.9688 124.3806 0)
 			(effects
 				(font
@@
 	(symbol
 		(lib_id "HW_template:Radar K-LC5-RFB-00C")
-		(at 247.65 111.76 0)
+		(at 245.11 116.84 0)
 		(unit 1)
 		(exclude_from_sim yes)
@@
 		(fields_autoplaced yes)
 		(property "Reference" "Y2"
-			(at 247.65 96.52 0)
+			(at 245.11 101.6 0)
 			(effects
 				(font
@@
 		)
 		(property "Value" "${SIM.PARAMS}"
-			(at 246.38 99.06 0)
+			(at 243.84 104.14 0)
 			(effects
 				(font
@@
 		)
 		(property "Footprint" "HW_template:Radar_K-LC5"
-			(at 246.38 125.73 0)
+			(at 243.84 130.81 0)
 			(effects
 				(font
@@
 		)
 		(property "Datasheet" "https://rfbeam.ch/product/k-lc5-radar-transceiver/"
-			(at 246.38 128.27 0)
+			(at 243.84 133.35 0)
 			(effects
 				(font
@@
 		)
 		(property "Description" ""
-			(at 247.65 111.76 0)
+			(at 245.11 116.84 0)
 			(effects
 				(font
@@
 		)
 		(property "Sim.Device" "SPICE"
-			(at 0 0 0)
+			(at -2.54 5.08 0)
 			(effects
 				(font
@@
 		)
 		(property "Sim.Params" "Radar K-LC5-RFB-00C"
-			(at 246.38 99.06 0)
+			(at 243.84 104.14 0)
 			(effects
 				(font
@@
 		)
 		(property "Sim.Pins" "1=1 2=2 3=3 4=4 5=5"
-			(at 0 0 0)
+			(at -2.54 5.08 0)
 			(effects
 				(font
@@
 	(symbol
 		(lib_id "power:GND")
-		(at 228.6 119.38 0)
+		(at 226.06 124.46 0)
 		(unit 1)
 		(exclude_from_sim no)
@@
 		(fields_autoplaced yes)
 		(property "Reference" "#PWR044"
-			(at 228.6 125.73 0)
+			(at 226.06 130.81 0)
 			(effects
 				(font
@@
 		)
 		(property "Value" "GND"
-			(at 228.6 124.46 0)
+			(at 226.06 129.54 0)
 			(effects
 				(font
@@
 		)
 		(property "Footprint" ""
-			(at 228.6 119.38 0)
+			(at 226.06 124.46 0)
 			(effects
 				(font
@@
 		)
 		(property "Datasheet" ""
-			(at 228.6 119.38 0)
+			(at 226.06 124.46 0)
 			(effects
 				(font
@@
 		)
 		(property "Description" "Power symbol creates a global label with name \"GND\" , ground"
-			(at 228.6 119.38 0)
+			(at 226.06 124.46 0)
 			(effects
 				(font
@@
 	(symbol
 		(lib_id "power:+3V0")
-		(at 228.6 104.14 0)
+		(at 226.06 109.22 0)
 		(unit 1)
 		(exclude_from_sim no)
@@
 		(dnp no)
 		(property "Reference" "#PWR043"
-			(at 228.6 107.95 0)
+			(at 226.06 113.03 0)
 			(effects
 				(font
@@
 		)
 		(property "Value" "+3V0"
-			(at 228.6 100.33 0)
+			(at 226.06 105.41 0)
 			(effects
 				(font
@@
 		)
 		(property "Footprint" ""
-			(at 228.6 104.14 0)
+			(at 226.06 109.22 0)
 			(effects
 				(font
@@
 		)
 		(property "Datasheet" ""
-			(at 228.6 104.14 0)
+			(at 226.06 109.22 0)
 			(effects
 				(font
@@
 		)
 		(property "Description" "Power symbol creates a global label with name \"+3V0\""
-			(at 228.6 104.14 0)
+			(at 226.06 109.22 0)
 			(effects
 				(font

Commit message: lol
Parts:
- removed C4: 100uF, Capacitor_SMD:C_1206_3216Metric_Pad1.33x1.80mm_HandSolder, symbol Device:C
- removed C6: 10uF, Capacitor_SMD:C_0805_2012Metric_Pad1.18x1.45mm_HandSolder, symbol Device:C
- removed C8, C9: 100nF, Capacitor_SMD:C_0805_2012Metric_Pad1.18x1.45mm_HandSolder, symbol Device:C
- removed J1: ${SIM.PARAMS}, Connector_USB:USB_Mini-B_Lumberg_2486_01_Horizontal, symbol Connector:USB_B_Mini
- removed LED1: LEDblue, LED_SMD:LED_1206_3216Metric_Pad1.42x1.75mm_HandSolder, symbol Device:LED
- removed LED2: LEDgreen, LED_SMD:LED_1206_3216Metric_Pad1.42x1.75mm_HandSolder, symbol Device:LED
- removed R10: 47, Resistor_SMD:R_0805_2012Metric_Pad1.20x1.40mm_HandSolder, symbol Device:R
- removed R12, R14: 100, Resistor_SMD:R_0805_2012Metric_Pad1.20x1.40mm_HandSolder, symbol Device:R
- removed R13: 1k, Resistor_SMD:R_0805_2012Metric_Pad1.20x1.40mm_HandSolder, symbol Device:R
- removed R9: 22, Resistor_SMD:R_0805_2012Metric_Pad1.20x1.40mm_HandSolder, symbol Device:R
- removed SD1: SD103AWS, Diode_SMD:D_SOD-323_HandSoldering, symbol Device:D_Schottky
- removed SW1: ${SIM.PARAMS}, Button_Switch_SMD:SW_SPST_PTS645, symbol Switch:SW_Push
- removed U3: SiP32508, Package_TO_SOT_SMD:TSOT-23-6_HandSoldering, symbol HW_template:SiP32508
- removed U5: ${SIM.PARAMS}, Package_TO_SOT_SMD:SOT-23, symbol Sensor_Magnetic:DRV5055A1xDBZxQ1
- removed U6: ${SIM.PARAMS}, HW_template:TO-92Flat_wide, symbol Sensor_Magnetic:DRV5055A1xLPGxQ1
- removed Y1: ${SIM.PARAMS}, Connector_PinHeader_2.54mm:PinHeader_1x06_P2.54mm_Vertical, symbol HW_template:OpenLog
- removed Y2: ${SIM.PARAMS}, HW_template:Radar_K-LC5, symbol HW_template:Radar K-LC5-RFB-00C
- added BT1: BH-18650-PC, BH-18650-PC:BAT_BH-18650-PC, symbol BH-18650-PC:BH-18650-PC
- added C23, C25, C26, C28, C29, C30: 10uF, Capacitor_SMD:C_0805_2012Metric_Pad1.18x1.45mm_HandSolder, symbol Device:C
- added C24: 10nF, Capacitor_SMD:C_0805_2012Metric_Pad1.18x1.45mm_HandSolder, symbol Device:C
- added C31: 1uF, Capacitor_SMD:C_0805_2012Metric_Pad1.18x1.45mm_HandSolder, symbol Device:C
- added CHARGE1: LEDcharge, LED_SMD:LED_1206_3216Metric_Pad1.42x1.75mm_HandSolder, symbol Device:LED
- added COMPLETE1: LEDcompl, LED_SMD:LED_1206_3216Metric_Pad1.42x1.75mm_HandSolder, symbol Device:LED
- added J1: Micro_SD_Card, Connector_Card:microSD_HC_Wuerth_693072010801, symbol Connector:Micro_SD_Card
- added J2: ${SIM.PARAMS}, Connector_USB:USB_Mini-B_Lumberg_2486_01_Horizontal, symbol Connector:USB_B_Mini
- added L1: 10 uH, Inductor_SMD:L_0805_2012Metric_Pad1.15x1.40mm_HandSolder, symbol Device:L
- added POWER1: LEDpower, LED_SMD:LED_1206_3216Metric_Pad1.42x1.75mm_HandSolder, symbol Device:LED
- added Q10, Q9: Si2319CDS, Package_TO_SOT_SMD:SOT-23, symbol Transistor_FET:Si2319CDS
- added Q4, Q5, Q6, Q7: BSS316N, Package_TO_SOT_SMD:SOT-23, symbol Transistor_FET:BSS138
- added R18, R19: 10kOhm, Resistor_SMD:R_0805_2012Metric_Pad1.20x1.40mm_HandSolder, symbol Device:R
- added R20, R21, R41, R42, R48: 1k, Resistor_SMD:R_0805_2012Metric_Pad1.20x1.40mm_HandSolder, symbol Device:R
- added R43: 30.1k, Resistor_SMD:R_0805_2012Metric_Pad1.20x1.40mm_HandSolder, symbol Device:R
- added R44: 330, Resistor_SMD:R_0805_2012Metric_Pad1.20x1.40mm_HandSolder, symbol Device:R
- added R45: 2.7k, Resistor_SMD:R_0805_2012Metric_Pad1.20x1.40mm_HandSolder, symbol Device:R
- added R46, R49, R50, R53, R54: 10k, Resistor_SMD:R_0805_2012Metric_Pad1.20x1.40mm_HandSolder, symbol Device:R
- added R47: 51k, Resistor_SMD:R_0805_2012Metric_Pad1.20x1.40mm_HandSolder, symbol Device:R
- added R51, R52: 100k, Resistor_SMD:R_0805_2012Metric_Pad1.20x1.40mm_HandSolder, symbol Device:R
- added SW1: SW_MEC_5G, Button_Switch_SMD:SW_SPST_EVQQ2, symbol Switch:SW_MEC_5G
- added TP4: ${SIM.PARAMS}, TestPoint:TestPoint_Loop_D2.60mm_Drill1.6mm_Beaded, symbol Connector:TestPoint
- added U1: LM2731XMF, Package_TO_SOT_SMD:SOT-23-5, symbol Regulator_Switching:LM2731XMF
- added U2: MCP73833-xxx-MF, Package_DFN_QFN:DFN-10-1EP_3x3mm_P0.5mm_EP1.58x2.35mm, symbol Battery_Management:MCP73833-xxx-MF
- added U3: AP9101CK, Package_TO_SOT_SMD:SOT-23-5, symbol Battery_Management:AP9101CK
- added Y4: ${SIM.PARAMS}, HW_template:Radar_K-LC5, symbol HW_template:Radar K-LC5-RFB-00C
Connections:
- net +3V0: now also J1.4 (VDD)
- net +5V: now also Q10.3 (D), R54.2
- net GND: now also C23.2, C24.2, C25.2, C29.1, C30.1, C31.2, J1.6 (VSS), J1.9 (SHIELD), J2.4 (ID), J2.5 (GND), J2.6 (Shield), Q4.2 (S), Q6.2 (S), Q7.2 (S), R19.1, R20.2, R46.2, R48.2, R49.1, R51.1, U1.2 (GND), U2.11 (EP), U2.5 (V_{SS}), U3.3 (VSS), Y4.4 (GND); no longer SD2.1 (K)
- net PE6: now also J1.7 (DAT0)
- net at U4.3 (VI): now also SD2.1 (K), C28.2, C29.2, Q9.2 (S), R43.2
- net at SD2.2 (A): now also L1.2, U1.1 (SW)
- net 3V3_INT renamed +3.3V
- net +3.3V: now also R18.2, R48.1, Y4.2 (VCC); no longer R17.1
- new net: BT1.N, C26.2, Q5.2 (S), R45.1
- new net: BT1.P, C26.1, L1.1, R44.2, R47.2, U1.5 (VIN), U2.10 (V_{BAT}), U2.9 (V_{BAT})
- new net: Q7.1 (G), R54.1, SW1.3 (B), SW1.4 (B)
- new net: C28.1, R43.1, R46.1, U1.3 (FB)
- new net: Q9.1 (G), R50.1, R51.2
- new net: POWER1.1 (K), R21.1
- new net: R21.2, U2.7 (~{PG})
- new net: CHARGE1.1 (K), R41.1
- new net: Q10.1 (G), Q7.3 (D), R52.2, R53.1
- new net: Q10.2 (S), Q9.3 (D), R53.2
- new net: R41.2, U2.4 (STAT2)
- new net: R45.2, U3.1 (VM)
- new net: C30.2, R44.1, U3.2 (VDD)
- new net: Q4.1 (G), U3.4 (DO)
- new net: Q5.1 (G), U3.5 (CO)
- new net: Q6.3 (D), R47.1, U1.4 (EN)
- new net: C31.1, R52.1, SW1.1 (A), SW1.2 (A)
- new net: R20.1, U2.8 (THERM)
- new net: R17.1, U2.6 (PROG)
- new net: COMPLETE1.1 (K), R42.1
- new net: R42.2, U2.3 (STAT1)
- new net: Q4.3 (D), Q5.3 (D)
- new net +1V65: C23.1, C24.1, R18.1, R19.2, TP4.1
- new net 5V: C25.1, CHARGE1.2 (A), COMPLETE1.2 (A), J2.1 (VBUS), POWER1.2 (A), Q6.1 (G), R49.2, R50.2, U2.1 (V_{DD}), U2.2 (V_{DD})
- new net IF_I: Y4.3 (IF_I)
- new net IF_Q: Y4.1 (IF_Q)
- new net PE2: J1.5 (CLK)
- new net PE4: J1.2 (DAT3/CD)
- new net PE5: J1.3 (CMD)
- no-connect marks 0 -> 2
Other:
- note removed: "Hall sensors can be used instead of coils. Choose SMD or THT version according to the direction of the lines of magnetic flux."
- note removed: "Linear 3.3V low drop regulator The 3V from the microcontroller board can also be used or the microcontroller can be feed by this regulator. Connect to correct supply nets or header pins."
- note removed: "Load switch Can be used to power on with pushbutton and power off via microcontroller. Connect to correct supply nets or header pins."
- note removed: "Miscellanneous components and subcircuits: Delete what is no used and copy components that are used several times."
- note removed: "Power Schottky"
- note removed: "Signal Schottky"
- note removed: "The OpenLog extension can be used for logging data onto an SD card"
- note removed: "The Radar sensor will be used in the project module 4"
- note removed: "USB connector might be useful for additional external supply"
- moved on the sheet: C7, LED3, Q1, R11, R15, R16, SD2, U4

Commit message: adasdasd
Parts:
- removed R16: 10, Resistor_SMD:R_0805_2012Metric_Pad1.20x1.40mm_HandSolder, symbol Device:R
- added CHARGE2: LEDcharge, LED_SMD:LED_1206_3216Metric_Pad1.42x1.75mm_HandSolder, symbol Device:LED
- added R55: 1k, Resistor_SMD:R_0805_2012Metric_Pad1.20x1.40mm_HandSolder, symbol Device:R
- added TP14, TP15, TP16, TP17, TP18, TP19, TP20: ~, TestPoint:TestPoint_Loop_D2.60mm_Drill1.6mm_Beaded, symbol Connector:TestPoint
Connections:
- net +3.3V: now also TP19.1
- net +5V: now also Q1.3 (D), TP14.1
- net 5V: now also TP17.1
- net Enable: now also CHARGE2.2 (A)
- net GND: now also R55.2
- net at BT1.P, C26.1, L1.1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: now also TP16.1
- net PA6: now reaches Q7.1 (G), R54.1, SW1.3 (B), SW1.4 (B)
- net at C28.2, C29.2, Q9.2 (S)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: now also TP18.1
- net at Q10.2 (S), Q9.3 (D), R53.2: now also TP15.1
- net at Q6.3 (D), R47.1, U1.4 (EN): now also TP20.1
- new net: CHARGE2.1 (K), R55.1

Commit message: PCB ORDERED
Parts:
- removed Q9: Si2319CDS, Package_TO_SOT_SMD:SOT-23, symbol Transistor_FET:Si2319CDS
- removed R50: 10k, Resistor_SMD:R_0805_2012Metric_Pad1.20x1.40mm_HandSolder, symbol Device:R
- removed R51: 100k, Resistor_SMD:R_0805_2012Metric_Pad1.20x1.40mm_HandSolder, symbol Device:R
- removed SW1: SW_MEC_5G, Button_Switch_SMD:SW_SPST_EVQQ2, symbol Switch:SW_MEC_5G
- removed TP15: ~, TestPoint:TestPoint_Loop_D2.60mm_Drill1.6mm_Beaded, symbol Connector:TestPoint
- added LS1: SMT-0827-S-HT-R, SMT-0827-S-HT-R:XDCR_SMT-0827-S-HT-R, symbol SMT-0827-S-HT-R:SMT-0827-S-HT-R
- added R16: 330, Resistor_SMD:R_0805_2012Metric_Pad1.20x1.40mm_HandSolder, symbol Device:R
- added SD3: SS13L, Diode_SMD:D_SMA, symbol Device:D_Schottky
- added SW1: SW_Push_Dual_x2, Button_Switch_SMD:SW_SPST_EVQQ2, symbol Switch:SW_Push_Dual_x2
- renumbered CHARGE1 to CRG1, COMPLETE1 to FULL1, POWER1 to PWR1
Connections:
- net +3V0 is gone; now on net +3.3V: J1.4 (VDD)
- net +5V: now also LS1.P; no longer Q1.3 (D)
- net 5V: now also SD3.2 (A)
- net Enable: no longer CHARGE2.2 (A), Q1.1 (G), R15.1
- net PA6: now also SW1.2 (D)
- net at C28.2, C29.2, R43.2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: now also Q10.2 (S), R53.2, SD3.1 (K)
- net fmcw_sig: now reaches Y4.5 (VCO_in)
- net at C31.1, R52.1: now also SW1.1 (C)
- new net: Q1.1 (G), R16.2
- new net: LS1.N, Q1.3 (D)
- new net LED_ON: CHARGE2.2 (A)
- new net PA8: R15.1, R16.1
Other:
- moved on the sheet: C31, C7, CHARGE2, Q1, Q10, Q7, R15, R48, R52, R53, R54, R55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
