File: HW_roggeluc_linortho/amplifier_filter_1channel.kicad_sch (KiCad schematic)
At the start: 6 parts, among them U7 MCP6002-xSN

Commit message: OPAMP ANTENNA
Parts:
- removed R18: 10k, Resistor_SMD:R_0805_2012Metric_Pad1.20x1.40mm_HandSolder, symbol Device:R
- removed R19, R21: 1k, Resistor_SMD:R_0805_2012Metric_Pad1.20x1.40mm_HandSolder, symbol Device:R
- removed R20: 12k, Resistor_SMD:R_0805_2012Metric_Pad1.20x1.40mm_HandSolder, symbol Device:R
- removed unit 1 of U7
- added C11, C12, C13, C14, C15, C16, C17, C18, C19: 100n, Capacitor_SMD:C_0805_2012Metric_Pad1.18x1.45mm_HandSolder, symbol Device:C
- added R26, R27, R28, R29, R30, R31, R32, R33, R34, R35, R36, R37: 1k, Resistor_SMD:R_0805_2012Metric_Pad1.20x1.40mm_HandSolder, symbol Device:R
- added U8: MCP6002-xSN, Package_SO:SOIC-8_3.9x4.9mm_P1.27mm, symbol Amplifier_Operational:MCP6002-xSN
- added Y3: ${SIM.PARAMS}, HW_template:Radar_K-LC5, symbol HW_template:Radar K-LC5-RFB-00C
Connections:
- net +3V0: now also C13.1, U8.8 (V+), Y3.2 (VCC)
- net GND: now also C12.1, C13.2, C19.1, R29.2, R31.2, R33.2, R36.2, U8.4 (V-), Y3.4 (GND)
- net at U7.5 (+): now also U7.1, R28.1
- net at U7.6 (-): now also C15.1, R31.1
- net out: no longer names the net of U7.7
- net out: now also R27.1, R30.1
- new net: C15.2, R30.2
- new net: C16.1, R33.1, U8.2 (-)
- new net: C16.2, R32.2
- new net: C11.2, R26.2, U7.3 (+)
- new net: C12.2, R27.2
- new net: R35.1, R37.1, U8.7
- new net: C18.2, R35.2
- new net: C18.1, R36.1, U8.6 (-)
- new net: C14.2, R28.2
- new net: R32.1, U8.1, U8.5 (+)
- new net: C17.2, R34.2, U8.3 (+)
- new net: C19.2, R37.2
- new net: C14.1, R29.1, U7.2 (-)
- new net PA5: Y3.5 (VCO_in)
Other:
- note added: "The Radar sensor will be used in the project module 4"
- note removed: "Use this template if two opamps are used for better amplification and filtering. As dual opamps are used, one channel only can be handled by this sheet."
- moved on the sheet: C10, U7C

Commit message: kek
Parts:
- removed Y3: ${SIM.PARAMS}, HW_template:Radar_K-LC5, symbol HW_template:Radar K-LC5-RFB-00C
- added C20, C21, C22: 100n, Capacitor_SMD:C_0805_2012Metric_Pad1.18x1.45mm_HandSolder, symbol Device:C
- added Q2, Q3: BSS316N, Package_TO_SOT_SMD:SOT-23, symbol Transistor_FET:BSS138
- added R38: 1k, Resistor_SMD:R_0805_2012Metric_Pad1.20x1.40mm_HandSolder, symbol Device:R
- added R39, R40: 10k, Resistor_SMD:R_0805_2012Metric_Pad1.20x1.40mm_HandSolder, symbol Device:R
- added TP10, TP11, TP12, TP13, TP8, TP9: ~, TestPoint:TestPoint_Loop_D2.60mm_Drill1.6mm_Beaded, symbol Connector:TestPoint
- added TP6: CH1, TestPoint:TestPoint_Loop_D2.60mm_Drill1.6mm_Beaded, symbol Connector:TestPoint
- added TP7: CH2, TestPoint:TestPoint_Loop_D2.60mm_Drill1.6mm_Beaded, symbol Connector:TestPoint
- added unit 2 of U7
Connections:
- net +3V0 is gone; now on net +3.3V: C10.1, C13.1, U7.8 (V+), U8.8 (V+)
- net GND: now also C20.1, Q2.2 (S), Q3.2 (S), R39.2, R40.2
- net at R27.1, R30.1: now also U7.7; no longer U7.7
- net at C15.2, R30.2: now also U7.6 (-)
- net at C16.1, R33.1: no longer U8.2 (-)
- net at C16.2, R32.2: now also U8.2 (-)
- net IF_I: now reaches C11.1
- net at C11.2, R26.2, U7.3 (+): now also TP10.1
- net ch1: now reaches C12.2, R27.2
- net ch1: now also C21.2, TP6.1
- net at C18.2, R35.2: now also U8.6 (-)
- net at C15.1, R31.1: no longer U7.6 (-)
- net at C18.1, R36.1: no longer U8.6 (-)
- net at R28.1, U7.1: now also TP9.1, U7.5 (+); no longer U7.5 (+)
- net at C14.2, R28.2: now also U7.2 (-)
- net at R32.1, U8.1, U8.5 (+): now also TP8.1
- net at C17.2, R34.2, U8.3 (+): now also TP11.1
- net ch2: now reaches C19.2, R37.2
- net ch2: now also C22.2, TP7.1
- net at C14.1, R29.1: no longer U7.2 (-)
- net +3.3V: now reaches R34.1
- net +3.3V: now also R26.1
- net IF_Q: now reaches C17.1
- new net: C21.1, Q2.3 (D)
- new net: C22.1, Q3.3 (D)
- new net bdw_en: Q2.1 (G), Q3.1 (G), R39.1, R40.1
- new net dac: R38.1, TP13.1
- new net fmcw_sig: C20.2, R38.2, TP12.1
Other:
- note added: "Saw-tooth signal for FMCW"
- note removed: "Some often used components are included here. Delete the components that are not used. Copy the components that are needed more than once."
- note removed: "The Radar sensor will be used in the project module 4"
- moved on the sheet: C10, C12, C13, C14, C15, C16, C17, C18, R27, R32, R33, R34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

Commit message: lol
Connections:
- net +3.3V: no longer R26.1, R34.1
- new net +1V65: R26.1, R34.1
Changed lines of the file:
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@@
 		(at 36.83 29.21 0)
 		(unit 1)
-		(exclude_from_sim yes)
+		(exclude_from_sim no)
 		(in_bom yes)
 		(on_board yes)
 		(dnp no)
-		(fields_autoplaced yes)
 		(property "Reference" "TP13"
-			(at 39.37 25.2729 0)
+			(at 34.544 23.876 0)
 			(effects
 				(font
@@
 		(at 110.49 50.8 0)
 		(unit 1)
-		(exclude_from_sim yes)
+		(exclude_from_sim no)
 		(in_bom yes)
 		(on_board yes)
@@
 		(at 257.81 50.8 0)
 		(unit 1)
-		(exclude_from_sim yes)
+		(exclude_from_sim no)
 		(in_bom yes)
 		(on_board yes)
@@
 		(at 149.86 53.34 0)
 		(unit 1)
-		(exclude_from_sim yes)
+		(exclude_from_sim no)
 		(in_bom yes)
 		(on_board yes)
@@
 	)
 	(symbol
-		(lib_id "Device:R")
-		(at 142.24 62.23 0)
+		(lib_id "power:+1V0")
+		(at 104.14 38.1 0)
 		(unit 1)
 		(exclude_from_sim no)
@@
 		(dnp no)
 		(fields_autoplaced yes)
-		(property "Reference" "R28"
-			(at 144.78 60.9599 0)
+		(property "Reference" "#PWR01"
+			(at 104.14 41.91 0)
 			(effects
 				(font
 					(size 1.27 1.27)
 				)
-				(justify left)
+				(hide yes)
 			)
 		)
-		(property "Value" "1k"
-			(at 144.78 63.4999 0)
+		(property "Value" "+1V65"
+			(at 104.14 33.02 0)
 			(effects
 				(font
 					(size 1.27 1.27)
 				)
-				(justify left)
 			)
 		)
-		(property "Footprint" "Resistor_SMD:R_0805_2012Metric_Pad1.20x1.40mm_HandSolder"
-			(at 140.462 62.23 90)
+		(property "Footprint" ""
+			(at 104.14 38.1 0)
 			(effects
 				(font
@@
 			)
 		)
-		(property "Datasheet" "~"
-			(at 142.24 62.23 0)
+		(property "Datasheet" ""
+			(at 104.14 38.1 0)
 			(effects
 				(font
@@
 			)
 		)
-		(property "Description" ""
-			(at 142.24 62.23 0)
+		(property "Description" "Power symbol creates a global label with name \"+1V0\""
+			(at 104.14 38.1 0)
 			(effects
 				(font
@@
 		(pin "1"
 		)
-		(pin "2"
-		)
 		(instances
-			(project "HW_roggeluc_linortho"
+			(project ""
 				(path "/1f276d59-ad9b-4e70-a842-f3b7e562eb9b/de01ffac-1f9d-4a03-9ae5-48822ed64956"
-					(reference "R28")
+					(reference "#PWR01")
 					(unit 1)
 				)
@@
 	)
 	(symbol
-		(lib_id "power:+3.3V")
-		(at 105.41 96.52 0)
+		(lib_id "Device:R")
+		(at 142.24 62.23 0)
 		(unit 1)
 		(exclude_from_sim no)
@@
 		(dnp no)
 		(fields_autoplaced yes)
-		(property "Reference" "#PWR015"
-			(at 105.41 100.33 0)
+		(property "Reference" "R28"
+			(at 144.78 60.9599 0)
 			(effects
 				(font
 					(size 1.27 1.27)
 				)
-				(hide yes)
+				(justify left)
 			)
 		)
-		(property "Value" "+3.3V"
-			(at 105.41 91.44 0)
+		(property "Value" "1k"
+			(at 144.78 63.4999 0)
 			(effects
 				(font
 					(size 1.27 1.27)
 				)
+				(justify left)
 			)
 		)
-		(property "Footprint" ""
-			(at 105.41 96.52 0)
+		(property "Footprint" "Resistor_SMD:R_0805_2012Metric_Pad1.20x1.40mm_HandSolder"
+			(at 140.462 62.23 90)
 			(effects
 				(font
@@
 			)
 		)
-		(property "Datasheet" ""
-			(at 105.41 96.52 0)
+		(property "Datasheet" "~"
+			(at 142.24 62.23 0)
 			(effects
 				(font
@@
 			)
 		)
-		(property "Description" "Power symbol creates a global label with name \"+3.3V\""
-			(at 105.41 96.52 0)
+		(property "Description" ""
+			(at 142.24 62.23 0)
 			(effects
 				(font
@@
 		(pin "1"
 		)
+		(pin "2"
+		)
 		(instances
 			(project "HW_roggeluc_linortho"
 				(path "/1f276d59-ad9b-4e70-a842-f3b7e562eb9b/de01ffac-1f9d-4a03-9ae5-48822ed64956"
-					(reference "#PWR015")
+					(reference "R28")
 					(unit 1)
 				)
@@
 	)
 	(symbol
-		(lib_id "power:+3.3V")
-		(at 104.14 38.1 0)
-		(unit 1)
-		(exclude_from_sim no)
-		(in_bom yes)
-		(on_board yes)
-		(dnp no)
-		(fields_autoplaced yes)
-		(property "Reference" "#PWR014"
-			(at 104.14 41.91 0)
-			(effects
-				(font
-					(size 1.27 1.27)
-				)
-				(hide yes)
-			)
-		)
-		(property "Value" "+3.3V"
-			(at 104.14 33.02 0)
-			(effects
-				(font
-					(size 1.27 1.27)
-				)
-			)
-		)
-		(property "Footprint" ""
-			(at 104.14 38.1 0)
-			(effects
-				(font
-					(size 1.27 1.27)
-				)
-				(hide yes)
-			)
-		)
-		(property "Datasheet" ""
-			(at 104.14 38.1 0)
-			(effects
-				(font
-					(size 1.27 1.27)
-				)
-				(hide yes)
-			)
-		)
-		(property "Description" "Power symbol creates a global label with name \"+3.3V\""
-			(at 104.14 38.1 0)
-			(effects
-				(font
-					(size 1.27 1.27)
-				)
-				(hide yes)
-			)
-		)
-		(pin "1"
-		)
-		(instances
-			(project "HW_roggeluc_linortho"
-				(path "/1f276d59-ad9b-4e70-a842-f3b7e562eb9b/de01ffac-1f9d-4a03-9ae5-48822ed64956"
-					(reference "#PWR014")
-					(unit 1)
-				)
-			)
-		)
-	)
-	(symbol
 		(lib_id "Amplifier_Operational:MCP6002-xSN")
 		(at 123.19 113.03 0)
@@
 		(at 149.86 110.49 0)
 		(unit 1)
-		(exclude_from_sim yes)
+		(exclude_from_sim no)
 		(in_bom yes)
 		(on_board yes)
@@
 	)
 	(symbol
+		(lib_id "power:+1V0")
+		(at 105.41 96.52 0)
+		(unit 1)
+		(exclude_from_sim no)
+		(in_bom yes)
+		(on_board yes)
+		(dnp no)
+		(fields_autoplaced yes)
+		(property "Reference" "#PWR02"
+			(at 105.41 100.33 0)
+			(effects
+				(font
+					(size 1.27 1.27)
+				)
+				(hide yes)
+			)
+		)
+		(property "Value" "+1V65"
+			(at 105.41 91.44 0)
+			(effects
+				(font
+					(size 1.27 1.27)
+				)
+			)
+		)
+		(property "Footprint" ""
+			(at 105.41 96.52 0)
+			(effects
+				(font
+					(size 1.27 1.27)
+				)
+				(hide yes)
+			)
+		)
+		(property "Datasheet" ""
+			(at 105.41 96.52 0)
+			(effects
+				(font
+					(size 1.27 1.27)
+				)
+				(hide yes)
+			)
+		)
+		(property "Description" "Power symbol creates a global label with name \"+1V0\""
+			(at 105.41 96.52 0)
+			(effects
+				(font
+					(size 1.27 1.27)
+				)
+				(hide yes)
+			)
+		)
+		(pin "1"
+		)
+		(instances
+			(project "HW_roggeluc_linortho"
+				(path "/1f276d59-ad9b-4e70-a842-f3b7e562eb9b/de01ffac-1f9d-4a03-9ae5-48822ed64956"
+					(reference "#PWR02")
+					(unit 1)
+				)
+			)
+		)
+	)
+	(symbol
 		(lib_id "Device:R")
 		(at 217.17 57.15 90)
@@
 		(at 257.81 114.3 0)
 		(unit 1)
-		(exclude_from_sim yes)
+		(exclude_from_sim no)
 		(in_bom yes)
 		(on_board yes)
@@
 		(at 111.76 110.49 0)
 		(unit 1)
-		(exclude_from_sim yes)
+		(exclude_from_sim no)
 		(in_bom yes)
 		(on_board yes)
@@
 		(at 60.96 29.21 0)
 		(unit 1)
-		(exclude_from_sim yes)
+		(exclude_from_sim no)
 		(in_bom yes)
 		(on_board yes)

Commit message: werteOPAMP
Parts:
- C11, C17: value 100n -> 1u
- C12, C19: value 100n -> 10n
- C14, C15, C16, C18, C21, C22: value 100n -> 10u
- R26, R34: value 1k -> 10k
- R28, R30, R32, R35: value 1k -> 30k
Changed lines of the file:
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@@
 			)
 		)
-		(property "Value" "1k"
+		(property "Value" "30k"
 			(at 194.31 63.4999 0)
 			(effects
@@
 			)
 		)
-		(property "Value" "100n"
+		(property "Value" "10u"
 			(at 147.32 132.0799 0)
 			(effects
@@
 			)
 		)
-		(property "Value" "100n"
+		(property "Value" "1u"
 			(at 93.98 46.99 90)
 			(effects
@@
 			)
 		)
-		(property "Value" "100n"
+		(property "Value" "10n"
 			(at 261.62 68.5799 0)
 			(effects
@@
 			)
 		)
-		(property "Value" "1k"
+		(property "Value" "30k"
 			(at 195.58 121.9199 0)
 			(effects
@@
 			)
 		)
-		(property "Value" "100n"
+		(property "Value" "10u"
 			(at 195.58 74.9299 0)
 			(effects
@@
 			)
 		)
-		(property "Value" "1k"
+		(property "Value" "30k"
 			(at 144.78 63.4999 0)
 			(effects
@@
 			)
 		)
-		(property "Value" "1k"
+		(property "Value" "30k"
 			(at 146.05 120.6499 0)
 			(effects
@@
 			)
 		)
-		(property "Value" "100n"
+		(property "Value" "10u"
 			(at 246.38 68.5799 0)
 			(effects
@@
 			)
 		)
-		(property "Value" "100n"
+		(property "Value" "10u"
 			(at 146.05 76.1999 0)
 			(effects
@@
 			)
 		)
-		(property "Value" "100n"
+		(property "Value" "10n"
 			(at 261.62 126.9999 0)
 			(effects
@@
 			)
 		)
-		(property "Value" "1k"
+		(property "Value" "10k"
 			(at 107.95 104.1399 0)
 			(effects
@@
 			)
 		)
-		(property "Value" "100n"
+		(property "Value" "10u"
 			(at 246.38 126.9999 0)
 			(effects
@@
 			)
 		)
-		(property "Value" "100n"
+		(property "Value" "10u"
 			(at 196.85 133.3499 0)
 			(effects
@@
 			)
 		)
-		(property "Value" "100n"
+		(property "Value" "1u"
 			(at 95.25 105.41 90)
 			(effects
@@
 			)
 		)
-		(property "Value" "1k"
+		(property "Value" "10k"
 			(at 106.68 45.7199 0)
 			(effects

Commit message: wydxgh
Parts:
- R26, R34: value 10k -> 11k
Changed lines of the file:
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@@
 			)
 		)
-		(property "Value" "10k"
+		(property "Value" "11k"
 			(at 107.95 104.1399 0)
 			(effects
@@
 			)
 		)
-		(property "Value" "10k"
+		(property "Value" "11k"
 			(at 106.68 45.7199 0)
 			(effects
